Commit message: Add KR10 R1100-2 visual meshes

File: kuka_kr10_support/urdf/kr10r1100_2_macro.xacro (robot description, xacro)
@@ -7,5 +7,5 @@
         <origin xyz="0 0 0" rpy="0 0 0"/>
         <geometry>
-          <mesh filename="package://kuka_kr10_support/meshes/kr10r1100sixx/visual/base_link.stl" />
+          <mesh filename="package://kuka_kr10_support/meshes/kr10r1100_2/visual/base_link.stl" />
         </geometry>
         <xacro:material_kuka_black />
@@ -22,5 +22,5 @@
         <origin xyz="0 0 0" rpy="0 0 0"/>
         <geometry>
-          <mesh filename="package://kuka_kr10_support/meshes/kr10r1100sixx/visual/link_1.stl" />
+          <mesh filename="package://kuka_kr10_support/meshes/kr10r1100_2/visual/link_1.stl" />
         </geometry>
         <xacro:material_kuka_orange />
@@ -37,5 +37,5 @@
         <origin xyz="0 0 0" rpy="0 0 0"/>
         <geometry>
-          <mesh filename="package://kuka_kr10_support/meshes/kr10r1100sixx/visual/link_2.stl"/>
+          <mesh filename="package://kuka_kr10_support/meshes/kr10r1100_2/visual/link_2.stl"/>
         </geometry>
         <xacro:material_kuka_orange />
@@ -52,5 +52,5 @@
         <origin xyz="0 0 0" rpy="0 0 0"/>
         <geometry>
-          <mesh filename="package://kuka_kr10_support/meshes/kr10r1100sixx/visual/link_3.stl" />
+          <mesh filename="package://kuka_kr10_support/meshes/kr10r1100_2/visual/link_3.stl" />
         </geometry>
         <xacro:material_kuka_orange />
@@ -67,5 +67,5 @@
         <origin xyz="0 0 0" rpy="0 0 0"/>
         <geometry>
-          <mesh filename="package://kuka_kr10_support/meshes/kr10r1100sixx/visual/link_4.stl" />
+          <mesh filename="package://kuka_kr10_support/meshes/kr10r1100_2/visual/link_4.stl" />
         </geometry>
         <xacro:material_kuka_orange />
@@ -82,5 +82,5 @@
         <origin xyz="0 0 0" rpy="0 0 0"/>
         <geometry>
-          <mesh filename="package://kuka_kr10_support/meshes/kr10r1100sixx/visual/link_5.stl" />
+          <mesh filename="package://kuka_kr10_support/meshes/kr10r1100_2/visual/link_5.stl" />
         </geometry>
         <xacro:material_kuka_orange />
@@ -97,5 +97,5 @@
         <origin xyz="0 0 0" rpy="0 0 0"/>
         <geometry>
-          <mesh filename="package://kuka_kr10_support/meshes/kr10r1100sixx/visual/link_6.stl" />
+          <mesh filename="package://kuka_kr10_support/meshes/kr10r1100_2/visual/link_6.stl" />
         </geometry>
         <xacro:material_kuka_pedestal />
